File: manually/manually.kicad_pcb (KiCad board)
At the start: 2 copper layers, 0 parts

Commit message: Tidy up a bit
Parts:
- added Z**: 3.5A-lap-pad, Library:3.5A-lap-pad, F.Cu at (68.3, 159.4)
- added Z**: 3.5A-lap-pad, Library:3.5A-lap-pad, B.Cu at (65.3, 111.8)
- added Z**1: 3.5A-lap-pad, Library:3.5A-lap-pad, F.Cu at (70.2, 159.4)
- added Z**10: 3.5A-lap-pad, Library:3.5A-lap-pad, B.Cu at (74.9, 111.8)
- added Z**100: 3.5A-lap-pad, Library:3.5A-lap-pad, B.Cu at (161.3, 111.8)
- added Z**101: 3.5A-lap-pad, Library:3.5A-lap-pad, F.Cu at (166.2, 159.4)
- added Z**102: 3.5A-lap-pad, Library:3.5A-lap-pad, B.Cu at (163.2, 111.8)
- added Z**11: 3.5A-lap-pad, Library:3.5A-lap-pad, F.Cu at (79.8, 159.4)
- added Z**12: 3.5A-lap-pad, Library:3.5A-lap-pad, B.Cu at (76.8, 111.8)
- added Z**13: 3.5A-lap-pad, Library:3.5A-lap-pad, F.Cu at (81.7, 159.4)
- added Z**14: 3.5A-lap-pad, Library:3.5A-lap-pad, B.Cu at (78.8, 111.8)
- added Z**15: 3.5A-lap-pad, Library:3.5A-lap-pad, F.Cu at (83.6, 159.4)
- added Z**16: 3.5A-lap-pad, Library:3.5A-lap-pad, B.Cu at (80.7, 111.8)
- added Z**17: 3.5A-lap-pad, Library:3.5A-lap-pad, F.Cu at (85.6, 159.4)
- added Z**18: 3.5A-lap-pad, Library:3.5A-lap-pad, B.Cu at (82.6, 111.8)
- added Z**19: 3.5A-lap-pad, Library:3.5A-lap-pad, F.Cu at (87.5, 159.4)
- added Z**2: 3.5A-lap-pad, Library:3.5A-lap-pad, B.Cu at (67.2, 111.8)
- added Z**20: 3.5A-lap-pad, Library:3.5A-lap-pad, B.Cu at (84.5, 111.8)
- added Z**21: 3.5A-lap-pad, Library:3.5A-lap-pad, F.Cu at (89.4, 159.4)
- added Z**22: 3.5A-lap-pad, Library:3.5A-lap-pad, B.Cu at (86.5, 111.8)
- added Z**23: 3.5A-lap-pad, Library:3.5A-lap-pad, F.Cu at (91.3, 159.4)
- added Z**24: 3.5A-lap-pad, Library:3.5A-lap-pad, B.Cu at (88.4, 111.8)
- added Z**25: 3.5A-lap-pad, Library:3.5A-lap-pad, F.Cu at (93.2, 159.4)
- added Z**26: 3.5A-lap-pad, Library:3.5A-lap-pad, B.Cu at (90.3, 111.8)
- added Z**27: 3.5A-lap-pad, Library:3.5A-lap-pad, F.Cu at (95.2, 159.4)
- added Z**28: 3.5A-lap-pad, Library:3.5A-lap-pad, B.Cu at (92.2, 111.8)
- added Z**29: 3.5A-lap-pad, Library:3.5A-lap-pad, F.Cu at (97.1, 159.4)
- added Z**3: 3.5A-lap-pad, Library:3.5A-lap-pad, F.Cu at (72.1, 159.4)
- added Z**30: 3.5A-lap-pad, Library:3.5A-lap-pad, B.Cu at (94.1, 111.8)
- added Z**31: 3.5A-lap-pad, Library:3.5A-lap-pad, F.Cu at (99.0, 159.4)
- added Z**32: 3.5A-lap-pad, Library:3.5A-lap-pad, B.Cu at (96.0, 111.8)
- added Z**33: 3.5A-lap-pad, Library:3.5A-lap-pad, F.Cu at (100.9, 159.4)
- added Z**34: 3.5A-lap-pad, Library:3.5A-lap-pad, B.Cu at (98.0, 111.8)
- added Z**35: 3.5A-lap-pad, Library:3.5A-lap-pad, F.Cu at (102.8, 159.4)
- added Z**36: 3.5A-lap-pad, Library:3.5A-lap-pad, B.Cu at (99.9, 111.8)
- added Z**37: 3.5A-lap-pad, Library:3.5A-lap-pad, F.Cu at (104.8, 159.4)
- added Z**38: 3.5A-lap-pad, Library:3.5A-lap-pad, B.Cu at (101.8, 111.8)
- added Z**39: 3.5A-lap-pad, Library:3.5A-lap-pad, F.Cu at (106.7, 159.4)
- added Z**4: 3.5A-lap-pad, Library:3.5A-lap-pad, B.Cu at (69.2, 111.8)
- added Z**40: 3.5A-lap-pad, Library:3.5A-lap-pad, B.Cu at (103.7, 111.8)
- added Z**41: 3.5A-lap-pad, Library:3.5A-lap-pad, F.Cu at (108.6, 159.4)
- added Z**42: 3.5A-lap-pad, Library:3.5A-lap-pad, B.Cu at (105.7, 111.8)
- added Z**43: 3.5A-lap-pad, Library:3.5A-lap-pad, F.Cu at (110.5, 159.4)
- added Z**44: 3.5A-lap-pad, Library:3.5A-lap-pad, B.Cu at (107.6, 111.8)
- added Z**45: 3.5A-lap-pad, Library:3.5A-lap-pad, F.Cu at (112.4, 159.4)
- added Z**46: 3.5A-lap-pad, Library:3.5A-lap-pad, B.Cu at (109.5, 111.8)
- added Z**47: 3.5A-lap-pad, Library:3.5A-lap-pad, F.Cu at (114.4, 159.4)
- added Z**48: 3.5A-lap-pad, Library:3.5A-lap-pad, B.Cu at (111.4, 111.8)
- added Z**49: 3.5A-lap-pad, Library:3.5A-lap-pad, F.Cu at (116.3, 159.4)
- added Z**5: 3.5A-lap-pad, Library:3.5A-lap-pad, F.Cu at (74.0, 159.4)
- added Z**50: 3.5A-lap-pad, Library:3.5A-lap-pad, B.Cu at (113.3, 111.8)
- added Z**51: 3.5A-lap-pad, Library:3.5A-lap-pad, F.Cu at (118.2, 159.4)
- added Z**52: 3.5A-lap-pad, Library:3.5A-lap-pad, B.Cu at (115.2, 111.8)
- added Z**53: 3.5A-lap-pad, Library:3.5A-lap-pad, F.Cu at (120.1, 159.4)
- added Z**54: 3.5A-lap-pad, Library:3.5A-lap-pad, B.Cu at (117.2, 111.8)
- added Z**55: 3.5A-lap-pad, Library:3.5A-lap-pad, F.Cu at (122.0, 159.4)
- added Z**56: 3.5A-lap-pad, Library:3.5A-lap-pad, B.Cu at (119.1, 111.8)
- added Z**57: 3.5A-lap-pad, Library:3.5A-lap-pad, F.Cu at (124.0, 159.4)
- added Z**58: 3.5A-lap-pad, Library:3.5A-lap-pad, B.Cu at (121.0, 111.8)
- added Z**59: 3.5A-lap-pad, Library:3.5A-lap-pad, F.Cu at (125.9, 159.4)
- added Z**6: 3.5A-lap-pad, Library:3.5A-lap-pad, B.Cu at (71.1, 111.8)
- added Z**60: 3.5A-lap-pad, Library:3.5A-lap-pad, B.Cu at (122.9, 111.8)
- added Z**61: 3.5A-lap-pad, Library:3.5A-lap-pad, F.Cu at (127.8, 159.4)
- added Z**62: 3.5A-lap-pad, Library:3.5A-lap-pad, B.Cu at (124.8, 111.8)
- added Z**63: 3.5A-lap-pad, Library:3.5A-lap-pad, F.Cu at (129.7, 159.4)
- added Z**64: 3.5A-lap-pad, Library:3.5A-lap-pad, B.Cu at (126.8, 111.8)
- added Z**65: 3.5A-lap-pad, Library:3.5A-lap-pad, F.Cu at (131.6, 159.4)
- added Z**66: 3.5A-lap-pad, Library:3.5A-lap-pad, B.Cu at (128.7, 111.8)
- added Z**67: 3.5A-lap-pad, Library:3.5A-lap-pad, F.Cu at (133.6, 159.4)
- added Z**68: 3.5A-lap-pad, Library:3.5A-lap-pad, B.Cu at (130.6, 111.8)
- added Z**69: 3.5A-lap-pad, Library:3.5A-lap-pad, F.Cu at (135.5, 159.4)
- added Z**7: 3.5A-lap-pad, Library:3.5A-lap-pad, F.Cu at (76.0, 159.4)
- added Z**70: 3.5A-lap-pad, Library:3.5A-lap-pad, B.Cu at (132.5, 111.8)
- added Z**71: 3.5A-lap-pad, Library:3.5A-lap-pad, F.Cu at (137.4, 159.4)
- added Z**72: 3.5A-lap-pad, Library:3.5A-lap-pad, B.Cu at (134.4, 111.8)
- added Z**73: 3.5A-lap-pad, Library:3.5A-lap-pad, F.Cu at (139.3, 159.4)
- added Z**74: 3.5A-lap-pad, Library:3.5A-lap-pad, B.Cu at (136.4, 111.8)
- added Z**75: 3.5A-lap-pad, Library:3.5A-lap-pad, F.Cu at (141.2, 159.4)
- added Z**76: 3.5A-lap-pad, Library:3.5A-lap-pad, B.Cu at (138.3, 111.8)
- added Z**77: 3.5A-lap-pad, Library:3.5A-lap-pad, F.Cu at (143.2, 159.4)
- added Z**78: 3.5A-lap-pad, Library:3.5A-lap-pad, B.Cu at (140.2, 111.8)
- added Z**79: 3.5A-lap-pad, Library:3.5A-lap-pad, F.Cu at (145.1, 159.4)
- added Z**8: 3.5A-lap-pad, Library:3.5A-lap-pad, B.Cu at (73.0, 111.8)
- added Z**80: 3.5A-lap-pad, Library:3.5A-lap-pad, B.Cu at (142.1, 111.8)
- added Z**81: 3.5A-lap-pad, Library:3.5A-lap-pad, F.Cu at (147.0, 159.4)
- added Z**82: 3.5A-lap-pad, Library:3.5A-lap-pad, B.Cu at (144.1, 111.8)
- added Z**83: 3.5A-lap-pad, Library:3.5A-lap-pad, F.Cu at (148.9, 159.4)
- added Z**84: 3.5A-lap-pad, Library:3.5A-lap-pad, B.Cu at (146.0, 111.8)
- added Z**85: 3.5A-lap-pad, Library:3.5A-lap-pad, F.Cu at (150.8, 159.4)
- added Z**86: 3.5A-lap-pad, Library:3.5A-lap-pad, B.Cu at (147.9, 111.8)
- added Z**87: 3.5A-lap-pad, Library:3.5A-lap-pad, F.Cu at (152.8, 159.4)
- added Z**88: 3.5A-lap-pad, Library:3.5A-lap-pad, B.Cu at (149.8, 111.8)
- added Z**89: 3.5A-lap-pad, Library:3.5A-lap-pad, F.Cu at (154.7, 159.4)
- added Z**9: 3.5A-lap-pad, Library:3.5A-lap-pad, F.Cu at (77.9, 159.4)
- added Z**90: 3.5A-lap-pad, Library:3.5A-lap-pad, B.Cu at (151.7, 111.8)
- added Z**91: 3.5A-lap-pad, Library:3.5A-lap-pad, F.Cu at (156.6, 159.4)
- added Z**92: 3.5A-lap-pad, Library:3.5A-lap-pad, B.Cu at (153.7, 111.8)
- added Z**93: 3.5A-lap-pad, Library:3.5A-lap-pad, F.Cu at (158.5, 159.4)
- added Z**94: 3.5A-lap-pad, Library:3.5A-lap-pad, B.Cu at (155.6, 111.8)
- added Z**95: 3.5A-lap-pad, Library:3.5A-lap-pad, F.Cu at (160.4, 159.4)
- added Z**96: 3.5A-lap-pad, Library:3.5A-lap-pad, B.Cu at (157.5, 111.8)
- added Z**97: 3.5A-lap-pad, Library:3.5A-lap-pad, F.Cu at (162.4, 159.4)
- added Z**98: 3.5A-lap-pad, Library:3.5A-lap-pad, B.Cu at (159.4, 111.8)
- added Z**99: 3.5A-lap-pad, Library:3.5A-lap-pad, F.Cu at (164.3, 159.4)
Routing:
- net (no net): track 55.0 -> 0.00 mm
- net w: vias 0 -> 416
- added copper zone on B.Cu, net w
- added copper zone on F.Cu, net w
Other:
- board outline added: 102.8 x 54.6 mm
